File: main-board.kicad_sch (KiCad schematic)
At the start: 15 parts

Commit message: Repo update
Parts:
- added D1, D2, D3, D4, D5, D6, D7, D8, D9: 1N4007, Diode_THT:D_DO-41_SOD81_P10.16mm_Horizontal, symbol Diode:1N4007
- added Q1: IRF4905, Package_TO_SOT_THT:TO-220-3_Vertical, symbol Transistor_FET:IRF4905
- added R1: 100R, symbol Device:R
- T1, T2, T3, T4, T5, T6, T7, T8, T9: footprint (none) -> 8hp-tcu-pcb-library:2EDN7434FXTMA1
Connections:
- net GND: no longer U1. (Vin)
- net GNDPWR: now also D1.2 (A), D2.2 (A), D3.2 (A), D4.2 (A), D5.2 (A), D6.2 (A), D7.2 (A), D8.2 (A), D9.2 (A)
- net at T1.2 (D): now also D1.1 (K)
- net at T6.2 (D): now also D6.1 (K)
- net at T7.2 (D): now also D7.1 (K)
- net at T2.2 (D): now also D2.1 (K)
- net at T5.2 (D): now also D5.1 (K)
- net at U1. (Vin): now also U3.4 (INB)
- net at T3.2 (D): now also D3.1 (K)
- net at T8.2 (D): now also D8.1 (K)
- net at T4.2 (D): now also D4.1 (K)
- net at T9.2 (D): now also D9.1 (K)
Other:
- note added: "Is 1A sufficient for the flyback diode current rating?"
- note removed: "Consider eFuses in addition to/rather than P-channel FETs & TVS diodes for input protection"
- moved on the sheet: T1, T2, T3, T4, T5, T6, T7, T8, T9, U1, U2, U3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
